Commit message: Updated plots for quadrotor performance

File: hingeTestBed.URDF (robot description, URDF)
Before this commit: robot physics, 12 links, 11 joints
Links:
- link link0: mass .82 -> .92
- link link1: mass .82 -> .92
- link link2: mass .82 -> .92
- link link3: mass .82 -> .92
- link prop0: mass 0.02 -> .02
- link prop1: mass 0.02 -> .02
- link prop2: mass 0.02 -> .02
- link prop3: mass 0.02 -> .02
Joints:
- joint h0_joint: limit lower=-3.14 upper=3.14 effort=10000 velocity=10000 -> lower=-.5 upper=2 effort=10000 velocity=10000
- joint h1_joint: limit lower=-3.14 upper=3.14 effort=10000 velocity=10000 -> lower=-.5 upper=2 effort=10000 velocity=10000
- joint h2_joint: limit lower=-3.14 upper=3.14 effort=10000 velocity=10000 -> lower=-.5 upper=2 effort=10000 velocity=10000
