Commit message: Updated MIST URDF
Added Gen5 main wing

File: MIST.urdf (robot description, URDF)
Before this commit: robot physics, 4 links, 3 joints
Links:
- link link0: geometry collision box size=0.7 0.7 0.1; visual mesh filename=package://meshes/mist_mainwing.STL scale=0.001 0.001 0.001
- link link1: geometry collision box size=0.7 0.7 0.1; visual mesh filename=package://meshes/mist_mainwing.STL scale=0.001 0.001 0.001
- link link2: geometry collision box size=0.7 0.7 0.1; visual mesh filename=package://meshes/mist_mainwing.STL scale=0.001 0.001 0.001
- link link3: geometry collision box size=0.7 0.7 0.1; visual mesh filename=package://meshes/mist_mainwing.STL scale=0.001 0.001 0.001
Joints:
- joint h0_joint: limit lower=0 upper=1.57 effort=100 velocity=100 -> lower=0 upper=1.57079632679 effort=10 velocity=10; origin xyz=0 .55 0 rpy=0 0 0 -> xyz=0 .58 0 rpy=0 0 0
- joint h1_joint: limit lower=0 upper=1.57 effort=100 velocity=100 -> lower=0 upper=1.57079632679 effort=10 velocity=10; origin xyz=0 .55 0 rpy=0 0 0 -> xyz=0 .58 0 rpy=0 0 0
- joint h2_joint: limit lower=0 upper=1.57 effort=100 velocity=100 -> lower=0 upper=1.57079632679 effort=10 velocity=10; origin xyz=0 .55 0 rpy=0 0 0 -> xyz=0 .58 0 rpy=0 0 0

Commit message: Fixed hinge overshoot
*Changed joint control from VELOCITY to POSITION. Solves the overshoot when setting a high force. Currently behaves like the NomQ Gen5
*Adjusted the link collisions

File: MIST.urdf (robot description, URDF)
Before this commit: robot physics, 4 links, 3 joints
Joints:
- joint h0_joint: limit lower=0 upper=1.57079632679 effort=10 velocity=10 -> lower=0 upper=1.57079632679 effort=1 velocity=1
- joint h1_joint: limit lower=0 upper=1.57079632679 effort=10 velocity=10 -> lower=0 upper=1.57079632679 effort=1 velocity=1
- joint h2_joint: limit lower=0 upper=1.57079632679 effort=10 velocity=10 -> lower=0 upper=1.57079632679 effort=1 velocity=1

Commit message: Updated MIST URDF
*Added and trimmed control surfaces
*Played around with colors

File: MIST.urdf (robot description, URDF)
Before this commit: robot physics, 4 links, 3 joints
Links:
- added link ctrlsurf0, mass 20; visual mesh filename=package://meshes/mist_controlsurface.STL scale=0.001 0.001 0.001
- added link ctrlsurf1, mass 20; visual mesh filename=package://meshes/mist_controlsurface.STL scale=0.001 0.001 0.001
- added link ctrlsurf2, mass 20; visual mesh filename=package://meshes/mist_controlsurface.STL scale=0.001 0.001 0.001
- added link ctrlsurf3, mass 20; visual mesh filename=package://meshes/mist_controlsurface.STL scale=0.001 0.001 0.001
Joints:
- added joint link0_ctrlsurf0: type revolute, parent link0, child ctrlsurf0, origin xyz=-.003 0 -.08 rpy=0 0 0, axis 0 1 0, limit lower=-1.57079632679 upper=1.57079632679 effort=1 velocity=1
- added joint link1_ctrlsurf1: type revolute, parent link1, child ctrlsurf1, origin xyz=-.003 0 -.08 rpy=0 0 0, axis 0 1 0, limit lower=-1.57079632679 upper=1.57079632679 effort=1 velocity=1
- added joint link2_ctrlsurf2: type revolute, parent link2, child ctrlsurf2, origin xyz=-.003 0 -.08 rpy=0 0 0, axis 0 1 0, limit lower=-1.57079632679 upper=1.57079632679 effort=1 velocity=1
- added joint link3_ctrlsurf3: type revolute, parent link3, child ctrlsurf3, origin xyz=-.003 0 -.08 rpy=0 0 0, axis 0 1 0, limit lower=-1.57079632679 upper=1.57079632679 effort=1 velocity=1

Commit message: Feature: Low Poly Propellers

File: MIST.urdf (robot description, URDF)
Before this commit: robot physics, 8 links, 7 joints
Links:
- added link prop0, mass .1; visual mesh filename=package://meshes/propeller_ccw.dae scale=0.1 0.1 0.1
- added link prop1, mass .1; visual mesh filename=package://meshes/propeller_ccw.dae scale=0.1 0.1 0.1
- added link prop2, mass .1; visual mesh filename=package://meshes/propeller_ccw.dae scale=0.1 0.1 0.1
- added link prop3, mass .1; visual mesh filename=package://meshes/propeller_ccw.dae scale=0.1 0.1 0.1
Joints:
- added joint link0_prop0: type continuous, parent link0, child prop0, origin xyz=-.003 0 .185 rpy=0 0 0, axis 0 0 1, limit lower=-1.57079632679 upper=1.57079632679 effort=1 velocity=1
- added joint link1_prop1: type continuous, parent link1, child prop1, origin xyz=-.003 0 .185 rpy=0 0 0, axis 0 0 1, limit lower=-1.57079632679 upper=1.57079632679 effort=1 velocity=1
- added joint link2_prop2: type continuous, parent link2, child prop2, origin xyz=-.003 0 .185 rpy=0 0 0, axis 0 0 1, limit lower=-1.57079632679 upper=1.57079632679 effort=1 velocity=1
- added joint link3_prop3: type continuous, parent link3, child prop3, origin xyz=-.003 0 .185 rpy=0 0 0, axis 0 0 1, limit lower=-1.57079632679 upper=1.57079632679 effort=1 velocity=1

Commit message: Fixed: Propeller joint Ids
Made arrays for the joint ids as they are not sequential w.r.t. the URDF

File: MIST.urdf (robot description, URDF)
Before this commit: robot physics, 12 links, 11 joints
Joints:
- joint link0_prop0: limit lower=-1.57079632679 upper=1.57079632679 effort=1 velocity=1 -> (none); origin xyz=-.003 0 .185 rpy=0 0 0 -> xyz=-.003 .28 .185 rpy=0 0 0
- joint link1_prop1: limit lower=-1.57079632679 upper=1.57079632679 effort=1 velocity=1 -> (none); origin xyz=-.003 0 .185 rpy=0 0 0 -> xyz=-.003 .28 .185 rpy=0 0 0
- joint link2_prop2: limit lower=-1.57079632679 upper=1.57079632679 effort=1 velocity=1 -> (none); origin xyz=-.003 0 .185 rpy=0 0 0 -> xyz=-.003 .28 .185 rpy=0 0 0
- joint link3_prop3: limit lower=-1.57079632679 upper=1.57079632679 effort=1 velocity=1 -> (none); origin xyz=-.003 0 .185 rpy=0 0 0 -> xyz=-.003 .28 .185 rpy=0 0 0

Commit message: Working takeoff
Fixed the applyAction() indices for  applying a throttle. Links start at -1 index.

File: MIST.urdf (robot description, URDF)
Before this commit: robot physics, 12 links, 11 joints
Links:
- link ctrlsurf0: mass 20 -> 1
- link ctrlsurf1: mass 20 -> 1
- link ctrlsurf2: mass 20 -> 1
- link ctrlsurf3: mass 20 -> 1
Joints:
- joint h0_joint: child link0 -> link1; parent link1 -> link0
- joint h1_joint: child link1 -> link2; parent link2 -> link1
- joint h2_joint: child link2 -> link3; parent link3 -> link2

Commit message: Added simple motor torque
Added simple motor torque.

File: MIST.urdf (robot description, URDF)
Before this commit: robot physics, 12 links, 11 joints
Links:
- link link0: geometry collision box size=0.7 0.7 0.4; visual mesh filename=package://meshes/mist_mainwing.STL scale=0.001 0.001 0.001
- link link1: geometry collision box size=0.7 0.7 0.4; visual mesh filename=package://meshes/mist_mainwing.STL scale=0.001 0.001 0.001
- link link2: geometry collision box size=0.7 0.7 0.4; visual mesh filename=package://meshes/mist_mainwing.STL scale=0.001 0.001 0.001
- link link3: geometry collision box size=0.7 0.7 0.4; visual mesh filename=package://meshes/mist_mainwing.STL scale=0.001 0.001 0.001

Commit message: Added AGTree

File: MIST.urdf (robot description, URDF)
Before this commit: robot physics, 12 links, 11 joints
Links:
- link link0: geometry visual mesh filename=package://meshes/mist_mainwing.STL scale=0.001 0.001 0.001
- link link1: geometry visual mesh filename=package://meshes/mist_mainwing.STL scale=0.001 0.001 0.001
- link link2: geometry visual mesh filename=package://meshes/mist_mainwing.STL scale=0.001 0.001 0.001
- link link3: geometry visual mesh filename=package://meshes/mist_mainwing.STL scale=0.001 0.001 0.001

Commit message: Updated all masses
Updated wing, controlsurface, and propeller masses to appropriate values.

File: MIST.urdf (robot description, URDF)
Before this commit: robot physics, 12 links, 11 joints
Links:
- link ctrlsurf0: mass 1 -> .1
- link ctrlsurf1: mass 1 -> .1
- link ctrlsurf2: mass 1 -> .1
- link ctrlsurf3: mass 1 -> .1
- link link0: mass 20 -> 1
- link link1: mass 20 -> 1
- link link2: mass 20 -> 1
- link link3: mass 20 -> 1
- link prop0: mass .1 -> .02
- link prop1: mass .1 -> .02
- link prop2: mass .1 -> .02
- link prop3: mass .1 -> .02

Commit message: Updated URDF model

File: MIST.urdf (robot description, URDF)
Before this commit: robot physics, 12 links, 11 joints
Links:
- link ctrlsurf0: mass 1 -> .1
- link ctrlsurf1: mass 1 -> .1
- link ctrlsurf2: mass 1 -> .1
- link ctrlsurf3: mass 1 -> .1
- link link0: mass 20 -> 1; geometry collision box size=0.7 0.7 0.4; visual mesh filename=package://meshes/mist_mainwing.STL scale=0.001 0.001 0.001
- link link1: mass 20 -> 1; geometry collision box size=0.7 0.7 0.4; visual mesh filename=package://meshes/mist_mainwing.STL scale=0.001 0.001 0.001
- link link2: mass 20 -> 1; geometry collision box size=0.7 0.7 0.4; visual mesh filename=package://meshes/mist_mainwing.STL scale=0.001 0.001 0.001
- link link3: mass 20 -> 1; geometry collision box size=0.7 0.7 0.4; visual mesh filename=package://meshes/mist_mainwing.STL scale=0.001 0.001 0.001
- link prop0: mass .1 -> .02
- link prop1: mass .1 -> .02
- link prop2: mass .1 -> .02
- link prop3: mass .1 -> .02

Commit message: First iteration of wing aerodynamic forces

File: MIST.urdf (robot description, URDF)
Before this commit: robot physics, 12 links, 11 joints
Links:
- link link0: geometry collision box size=0.7 0.7 1.4; visual mesh filename=package://meshes/mist_mainwing.STL scale=0.001 0.001 0.001

Commit message: WIP - transformation with aerodynamics

File: MIST.urdf (robot description, URDF)
Before this commit: robot physics, 12 links, 11 joints
Links:
- link link0: geometry collision box size=0.7 0.7 0.4; visual mesh filename=package://meshes/mist_mainwing.STL scale=0.001 0.001 0.001

Commit message: Fixed sim issue, comments and some hyperparameters.

File: MIST.urdf (robot description, URDF)
Before this commit: robot physics, 12 links, 11 joints
Joints:
- joint h0_joint: limit lower=0 upper=1.57079632679 effort=1 velocity=1 -> lower=1.57079632679 upper=1.57079632679 effort=1 velocity=1
- joint h1_joint: limit lower=0 upper=1.57079632679 effort=1 velocity=1 -> lower=1.57079632679 upper=1.57079632679 effort=1 velocity=1
- joint h2_joint: limit lower=0 upper=1.57079632679 effort=1 velocity=1 -> lower=1.57079632679 upper=1.57079632679 effort=1 velocity=1

Commit message: Testing open-close hinge torques.

File: MIST.urdf (robot description, URDF)
Before this commit: robot physics, 12 links, 11 joints
Joints:
- joint h0_joint: limit lower=0 upper=1.57079632679 effort=1 velocity=1 -> lower=0 upper=2 effort=10000 velocity=10000
- joint h1_joint: limit lower=0 upper=1.57079632679 effort=1 velocity=1 -> lower=0 upper=1.6 effort=10000 velocity=10000
- joint h2_joint: limit lower=0 upper=1.57079632679 effort=1 velocity=1 -> lower=0 upper=2 effort=10000 velocity=10000

Commit message: Updated dynamics and routines
Working quadposition, fixedwing, and quad-fixedwing-quad

File: MIST.urdf (robot description, URDF)
Before this commit: robot physics, 12 links, 11 joints
Joints:
- joint link0_ctrlsurf0: origin xyz=-.003 0 -.08 rpy=0 0 0 -> xyz=-.003 .28 -.08 rpy=0 0 0
- joint link1_ctrlsurf1: origin xyz=-.003 0 -.08 rpy=0 0 0 -> xyz=-.003 .28 -.08 rpy=0 0 0
- joint link2_ctrlsurf2: origin xyz=-.003 0 -.08 rpy=0 0 0 -> xyz=-.003 .28 -.08 rpy=0 0 0
- joint link3_ctrlsurf3: origin xyz=-.003 0 -.08 rpy=0 0 0 -> xyz=-.003 .28 -.08 rpy=0 0 0

Commit message: Updated Routines

File: MIST.urdf (robot description, URDF)
Before this commit: robot physics, 12 links, 11 joints
Joints:
- joint h0_joint: limit lower=-3.14 upper=3.14 effort=10000 velocity=10000 -> lower=-.1 upper=3.14 effort=10000 velocity=10000
- joint h1_joint: limit lower=-3.14 upper=3.14 effort=10000 velocity=10000 -> lower=-.1 upper=3.14 effort=10000 velocity=10000
- joint h2_joint: limit lower=-3.14 upper=3.14 effort=10000 velocity=10000 -> lower=-.1 upper=3.14 effort=10000 velocity=10000
